Commit message: update nix1_v2 about ankle joint limit

File: nix1/urdf/nix1_v2_joint21_nomesh.urdf (robot description, URDF)
Before this commit: robot nix1, 22 links, 21 joints
Joints:
- joint left_ankle_pitch_joint: limit lower=-0.697 upper=0.697 effort=20 velocity=30 -> lower=-0.523 upper=0.523 effort=20 velocity=30
- joint left_ankle_roll_joint: limit lower=-0.348 upper=0.348 effort=20 velocity=30 -> lower=-0.262 upper=0.262 effort=20 velocity=30
- joint right_ankle_pitch_joint: limit lower=-0.697 upper=0.697 effort=20 velocity=30 -> lower=-0.523 upper=0.523 effort=20 velocity=30
- joint right_ankle_roll_joint: limit lower=-0.348 upper=0.348 effort=20 velocity=30 -> lower=-0.262 upper=0.262 effort=20 velocity=30
