Commit message: update some joint efforts

File: lus2/urdf/lus2_joint21.urdf (robot description, URDF)
Before this commit: robot lus2, 29 links, 28 joints
Joints:
- joint head_joint: limit lower=-1.3 upper=1.3 effort=20 velocity=20 -> lower=-1.3 upper=1.3 effort=17 velocity=87
- joint left_ankle_pitch_joint: limit lower=-1.0 upper=0.43 effort=200 velocity=20 -> lower=-1.0 upper=0.43 effort=100 velocity=14
- joint left_ankle_roll_joint: limit lower=-0.43 upper=0.43 effort=200 velocity=20 -> lower=-0.43 upper=0.43 effort=100 velocity=14
- joint left_elbow_joint: limit lower=-0.83 upper=1.57 effort=100 velocity=20 -> lower=-0.83 upper=1.57 effort=100 velocity=14
- joint left_shoulder_pitch_joint: limit lower=-3 upper=3 effort=100 velocity=20 -> lower=-3 upper=3 effort=100 velocity=14
- joint left_shoulder_roll_joint: limit lower=-0.12 upper=2.3 effort=100 velocity=20 -> lower=-0.12 upper=2.3 effort=100 velocity=14
- joint left_shoulder_yaw_joint: limit lower=-1.9 upper=1.9 effort=100 velocity=20 -> lower=-1.9 upper=1.9 effort=100 velocity=14
- joint left_wrist_pitch_joint: limit lower=-1.2 upper=1.2 effort=20 velocity=20 -> lower=-1.2 upper=1.2 effort=17 velocity=87
- joint left_wrist_roll_joint: limit lower=-1.2 upper=1.2 effort=20 velocity=20 -> lower=-1.2 upper=1.2 effort=17 velocity=87
- joint left_wrist_yaw_joint: limit lower=-2.3 upper=2.3 effort=20 velocity=20 -> lower=-2.3 upper=2.3 effort=17 velocity=87
- joint right_ankle_pitch_joint: limit lower=-1.0 upper=0.43 effort=200 velocity=20 -> lower=-1.0 upper=0.43 effort=100 velocity=14
- joint right_ankle_roll_joint: limit lower=-0.43 upper=0.43 effort=200 velocity=20 -> lower=-0.43 upper=0.43 effort=100 velocity=14
- joint right_elbow_joint: limit lower=-0.83 upper=1.57 effort=100 velocity=20 -> lower=-0.83 upper=1.57 effort=100 velocity=14
- joint right_shoulder_pitch_joint: limit lower=-3 upper=3 effort=100 velocity=20 -> lower=-3 upper=3 effort=100 velocity=14
- joint right_shoulder_roll_joint: limit lower=-2.3 upper=0.12 effort=100 velocity=20 -> lower=-2.3 upper=0.12 effort=100 velocity=14
- joint right_shoulder_yaw_joint: limit lower=-1.9 upper=1.9 effort=100 velocity=20 -> lower=-1.9 upper=1.9 effort=100 velocity=14
- joint right_wrist_pitch_joint: limit lower=-1.2 upper=1.2 effort=20 velocity=20 -> lower=-1.2 upper=1.2 effort=17 velocity=87
- joint right_wrist_roll_joint: limit lower=-1.2 upper=1.2 effort=20 velocity=20 -> lower=-1.2 upper=1.2 effort=17 velocity=87
- joint right_wrist_yaw_joint: limit lower=-2.3 upper=2.3 effort=20 velocity=20 -> lower=-2.3 upper=2.3 effort=17 velocity=87

Commit message: update joint vel

File: lus2/urdf/lus2_joint21.urdf (robot description, URDF)
Before this commit: robot lus2, 29 links, 28 joints
Joints:
- joint left_hip_pitch_joint: limit lower=-1.5 upper=1.5 effort=300 velocity=12 -> lower=-1.5 upper=1.5 effort=300 velocity=11
- joint left_hip_roll_joint: limit lower=-0.25 upper=2.8 effort=300 velocity=12 -> lower=-0.25 upper=2.8 effort=300 velocity=11
- joint left_hip_yaw_joint: limit lower=-1.2 upper=2.6 effort=300 velocity=12 -> lower=-1.2 upper=2.6 effort=300 velocity=11
- joint left_knee_joint: limit lower=0.0 upper=2.27 effort=300 velocity=12 -> lower=0.0 upper=2.27 effort=300 velocity=11
- joint right_hip_pitch_joint: limit lower=-1.5 upper=1.5 effort=300 velocity=12 -> lower=-1.5 upper=1.5 effort=300 velocity=11
- joint right_hip_roll_joint: limit lower=-2.8 upper=0.25 effort=300 velocity=12 -> lower=-2.8 upper=0.25 effort=300 velocity=11
- joint right_hip_yaw_joint: limit lower=-2.6 upper=1.2 effort=300 velocity=12 -> lower=-2.6 upper=1.2 effort=300 velocity=11
- joint right_knee_joint: limit lower=0.0 upper=2.27 effort=300 velocity=12 -> lower=0.0 upper=2.27 effort=300 velocity=11
- joint torso_joint: limit lower=-3 upper=3 effort=300 velocity=12 -> lower=-3 upper=3 effort=300 velocity=11

Commit message: update lus2 mass

File: lus2/urdf/lus2_joint21.urdf (robot description, URDF)
Before this commit: robot lus2, 29 links, 28 joints
Links:
- link left_elbow_link: mass 0.59309890 -> 8.1901234e-01
- link left_shoulder_pitch_link: mass 0.173114536540602 -> 3.0353084e-01
- link left_shoulder_roll_link: mass 0.364744656002893 -> 1.6480208e+00
- link left_shoulder_yaw_link: mass 1.12432170 -> 1.0475838e+00
- link left_wrist_pitch_link: mass 0.47109798 -> 7.3227634e-01
- link left_wrist_roll_link: geometry collision cylinder length=0.054 radius=0.035; collision mesh filename=../meshes/left_hand_link.STL scale=1 1 1
- link left_wrist_yaw_link: mass 0.36396026 -> 6.1426733e-01
- link right_elbow_link: mass 0.59309105 -> 8.1901252e-01
- link right_shoulder_pitch_link: mass 0.173115302786264 -> 3.0353084e-01
- link right_shoulder_roll_link: mass 0.364801949403457 -> 1.6480208e+00
- link right_shoulder_yaw_link: mass 1.12432180 -> 1.0475841e+00
- link right_wrist_pitch_link: mass 0.47109816 -> 7.3227634e-01
- link right_wrist_roll_link: geometry collision cylinder length=0.054 radius=0.035; collision mesh filename=../meshes/right_hand_link.STL scale=1 1 1
- link right_wrist_yaw_link: mass 0.36396026 -> 6.1426734e-01

File: lus2/urdf/lus2_joint25.urdf (robot description, URDF)
Before this commit: robot lus2, 29 links, 28 joints
Links:
- link left_ankle_roll_link: geometry collision box size=0.235 0.073 0.0143; collision sphere radius=0.005
- link left_elbow_link: mass 0.59309890 -> 8.1901234e-01
- link left_shoulder_pitch_link: mass 0.173114536540602 -> 3.0353084e-01
- link left_shoulder_roll_link: mass 0.364744656002893 -> 1.6480208e+00
- link left_shoulder_yaw_link: mass 1.12432170 -> 1.0475838e+00
- link left_wrist_pitch_link: mass 0.47109798 -> 7.3227634e-01
- link left_wrist_roll_link: geometry collision cylinder length=0.054 radius=0.035; collision mesh filename=../meshes/left_hand_link.STL scale=1 1 1
- link left_wrist_yaw_link: mass 0.36396026 -> 6.1426733e-01
- link right_ankle_roll_link: geometry collision box size=0.235 0.073 0.0143; collision sphere radius=0.005
- link right_elbow_link: mass 0.59309105 -> 8.1901252e-01
- link right_shoulder_pitch_link: mass 0.173115302786264 -> 3.0353084e-01
- link right_shoulder_roll_link: mass 0.364801949403457 -> 1.6480208e+00
- link right_shoulder_yaw_link: mass 1.12432180 -> 1.0475841e+00
- link right_wrist_pitch_link: mass 0.47109816 -> 7.3227634e-01
- link right_wrist_roll_link: geometry collision cylinder length=0.054 radius=0.035; collision mesh filename=../meshes/right_hand_link.STL scale=1 1 1
- link right_wrist_yaw_link: mass 0.36396026 -> 6.1426734e-01
Joints:
- joint head_joint: limit lower=-1.3 upper=1.3 effort=20 velocity=20 -> lower=-1.3 upper=1.3 effort=17 velocity=87
- joint left_ankle_pitch_joint: limit lower=-0.34 upper=0.17 effort=200 velocity=20 -> lower=-1.0 upper=0.43 effort=100 velocity=14
- joint left_ankle_roll_joint: limit lower=-0.26 upper=0.26 effort=200 velocity=20 -> lower=-0.43 upper=0.43 effort=100 velocity=14
- joint left_elbow_joint: limit lower=-0.83 upper=1.57 effort=100 velocity=20 -> lower=-0.83 upper=1.57 effort=100 velocity=14
- joint left_hip_pitch_joint: limit lower=-1.5 upper=1.5 effort=300 velocity=12 -> lower=-1.5 upper=1.5 effort=300 velocity=11
- joint left_hip_roll_joint: limit lower=-0.25 upper=2.8 effort=300 velocity=12 -> lower=-0.25 upper=2.8 effort=300 velocity=11
- joint left_hip_yaw_joint: limit lower=-1.2 upper=2.6 effort=300 velocity=12 -> lower=-1.2 upper=2.6 effort=300 velocity=11
- joint left_knee_joint: limit lower=0.0 upper=2.27 effort=300 velocity=12 -> lower=0.0 upper=2.27 effort=300 velocity=11
- joint left_shoulder_pitch_joint: limit lower=-3 upper=3 effort=100 velocity=20 -> lower=-3 upper=3 effort=100 velocity=14
- joint left_shoulder_roll_joint: limit lower=-0.12 upper=2.3 effort=100 velocity=20 -> lower=-0.12 upper=2.3 effort=100 velocity=14
- joint left_shoulder_yaw_joint: limit lower=-1.9 upper=1.9 effort=100 velocity=20 -> lower=-1.9 upper=1.9 effort=100 velocity=14
- joint left_wrist_pitch_joint: limit lower=-1.2 upper=1.2 effort=20 velocity=20 -> lower=-1.2 upper=1.2 effort=17 velocity=87
- joint left_wrist_roll_joint: limit lower=-1.2 upper=1.2 effort=20 velocity=20 -> lower=-1.2 upper=1.2 effort=17 velocity=87
- joint left_wrist_yaw_joint: limit lower=-2.3 upper=2.3 effort=20 velocity=20 -> lower=-2.3 upper=2.3 effort=17 velocity=87
- joint right_ankle_pitch_joint: limit lower=-0.34 upper=0.17 effort=200 velocity=20 -> lower=-1.0 upper=0.43 effort=100 velocity=14
- joint right_ankle_roll_joint: limit lower=-0.26 upper=0.26 effort=200 velocity=20 -> lower=-0.43 upper=0.43 effort=100 velocity=14
- joint right_elbow_joint: limit lower=-0.83 upper=1.57 effort=100 velocity=20 -> lower=-0.83 upper=1.57 effort=100 velocity=14
- joint right_hip_pitch_joint: limit lower=-1.5 upper=1.5 effort=300 velocity=12 -> lower=-1.5 upper=1.5 effort=300 velocity=11
- joint right_hip_roll_joint: limit lower=-2.8 upper=0.25 effort=300 velocity=12 -> lower=-2.8 upper=0.25 effort=300 velocity=11
- joint right_hip_yaw_joint: limit lower=-2.6 upper=1.2 effort=300 velocity=12 -> lower=-2.6 upper=1.2 effort=300 velocity=11
- joint right_knee_joint: limit lower=0.0 upper=2.27 effort=300 velocity=12 -> lower=0.0 upper=2.27 effort=300 velocity=11
- joint right_shoulder_pitch_joint: limit lower=-3 upper=3 effort=100 velocity=20 -> lower=-3 upper=3 effort=100 velocity=14
- joint right_shoulder_roll_joint: limit lower=-2.3 upper=0.12 effort=100 velocity=20 -> lower=-2.3 upper=0.12 effort=100 velocity=14
- joint right_shoulder_yaw_joint: limit lower=-1.9 upper=1.9 effort=100 velocity=20 -> lower=-1.9 upper=1.9 effort=100 velocity=14
- joint right_wrist_pitch_joint: limit lower=-1.2 upper=1.2 effort=20 velocity=20 -> lower=-1.2 upper=1.2 effort=17 velocity=87
- joint right_wrist_roll_joint: limit lower=-1.2 upper=1.2 effort=20 velocity=20 -> lower=-1.2 upper=1.2 effort=17 velocity=87
- joint right_wrist_yaw_joint: limit lower=-2.3 upper=2.3 effort=20 velocity=20 -> lower=-2.3 upper=2.3 effort=17 velocity=87
- joint torso_joint: limit lower=-3 upper=3 effort=300 velocity=12 -> lower=-3 upper=3 effort=300 velocity=11

File: lus2/urdf/lus2_joint27.urdf (robot description, URDF)
Before this commit: robot lus2, 29 links, 28 joints
Links:
- link left_ankle_roll_link: geometry collision box size=0.235 0.073 0.0143; collision sphere radius=0.005
- link left_elbow_link: mass 0.59309890 -> 8.1901234e-01
- link left_shoulder_pitch_link: mass 0.173114536540602 -> 3.0353084e-01
- link left_shoulder_roll_link: mass 0.364744656002893 -> 1.6480208e+00
- link left_shoulder_yaw_link: mass 1.12432170 -> 1.0475838e+00
- link left_wrist_pitch_link: mass 0.47109798 -> 7.3227634e-01
- link left_wrist_roll_link: geometry collision cylinder length=0.054 radius=0.035; collision mesh filename=../meshes/left_hand_link.STL scale=1 1 1
- link left_wrist_yaw_link: mass 0.36396026 -> 6.1426733e-01
- link right_ankle_roll_link: geometry collision box size=0.235 0.073 0.0143; collision sphere radius=0.005
- link right_elbow_link: mass 0.59309105 -> 8.1901252e-01
- link right_shoulder_pitch_link: mass 0.173115302786264 -> 3.0353084e-01
- link right_shoulder_roll_link: mass 0.364801949403457 -> 1.6480208e+00
- link right_shoulder_yaw_link: mass 1.12432180 -> 1.0475841e+00
- link right_wrist_pitch_link: mass 0.47109816 -> 7.3227634e-01
- link right_wrist_roll_link: geometry collision cylinder length=0.054 radius=0.035; collision mesh filename=../meshes/right_hand_link.STL scale=1 1 1
- link right_wrist_yaw_link: mass 0.36396026 -> 6.1426734e-01
Joints:
- joint head_joint: limit lower=-1.3 upper=1.3 effort=20 velocity=20 -> lower=-1.3 upper=1.3 effort=17 velocity=87
- joint left_ankle_pitch_joint: limit lower=-1.0 upper=0.43 effort=200 velocity=20 -> lower=-1.0 upper=0.43 effort=100 velocity=14
- joint left_ankle_roll_joint: limit lower=-0.43 upper=0.43 effort=200 velocity=20 -> lower=-0.43 upper=0.43 effort=100 velocity=14
- joint left_elbow_joint: limit lower=-0.83 upper=1.57 effort=100 velocity=20 -> lower=-0.83 upper=1.57 effort=100 velocity=14
- joint left_hip_pitch_joint: limit lower=-1.5 upper=1.5 effort=300 velocity=12 -> lower=-1.5 upper=1.5 effort=300 velocity=11
- joint left_hip_roll_joint: limit lower=-0.25 upper=2.8 effort=300 velocity=12 -> lower=-0.25 upper=2.8 effort=300 velocity=11
- joint left_hip_yaw_joint: limit lower=-1.2 upper=2.6 effort=300 velocity=12 -> lower=-1.2 upper=2.6 effort=300 velocity=11
- joint left_knee_joint: limit lower=0.0 upper=2.27 effort=300 velocity=12 -> lower=0.0 upper=2.27 effort=300 velocity=11
- joint left_shoulder_pitch_joint: limit lower=-3 upper=3 effort=100 velocity=20 -> lower=-3 upper=3 effort=100 velocity=14
- joint left_shoulder_roll_joint: limit lower=-0.12 upper=2.3 effort=100 velocity=20 -> lower=-0.12 upper=2.3 effort=100 velocity=14
- joint left_shoulder_yaw_joint: limit lower=-1.9 upper=1.9 effort=100 velocity=20 -> lower=-1.9 upper=1.9 effort=100 velocity=14
- joint left_wrist_pitch_joint: limit lower=-1.2 upper=1.2 effort=20 velocity=20 -> lower=-1.2 upper=1.2 effort=17 velocity=87
- joint left_wrist_roll_joint: limit lower=-1.2 upper=1.2 effort=20 velocity=20 -> lower=-1.2 upper=1.2 effort=17 velocity=87
- joint left_wrist_yaw_joint: limit lower=-2.3 upper=2.3 effort=20 velocity=20 -> lower=-2.3 upper=2.3 effort=17 velocity=87
- joint right_ankle_pitch_joint: limit lower=-1.0 upper=0.43 effort=200 velocity=20 -> lower=-1.0 upper=0.43 effort=100 velocity=14
- joint right_ankle_roll_joint: limit lower=-0.43 upper=0.43 effort=200 velocity=20 -> lower=-0.43 upper=0.43 effort=100 velocity=14
- joint right_elbow_joint: limit lower=-0.83 upper=1.57 effort=100 velocity=20 -> lower=-0.83 upper=1.57 effort=100 velocity=14
- joint right_hip_pitch_joint: limit lower=-1.5 upper=1.5 effort=300 velocity=12 -> lower=-1.5 upper=1.5 effort=300 velocity=11
- joint right_hip_roll_joint: limit lower=-2.8 upper=0.25 effort=300 velocity=12 -> lower=-2.8 upper=0.25 effort=300 velocity=11
- joint right_hip_yaw_joint: limit lower=-2.6 upper=1.2 effort=300 velocity=12 -> lower=-2.6 upper=1.2 effort=300 velocity=11
- joint right_knee_joint: limit lower=0.0 upper=2.27 effort=300 velocity=12 -> lower=0.0 upper=2.27 effort=300 velocity=11
- joint right_shoulder_pitch_joint: limit lower=-3 upper=3 effort=100 velocity=20 -> lower=-3 upper=3 effort=100 velocity=14
- joint right_shoulder_roll_joint: limit lower=-2.3 upper=0.12 effort=100 velocity=20 -> lower=-2.3 upper=0.12 effort=100 velocity=14
- joint right_shoulder_yaw_joint: limit lower=-1.9 upper=1.9 effort=100 velocity=20 -> lower=-1.9 upper=1.9 effort=100 velocity=14
- joint right_wrist_pitch_joint: limit lower=-1.2 upper=1.2 effort=20 velocity=20 -> lower=-1.2 upper=1.2 effort=17 velocity=87
- joint right_wrist_roll_joint: limit lower=-1.2 upper=1.2 effort=20 velocity=20 -> lower=-1.2 upper=1.2 effort=17 velocity=87
- joint right_wrist_yaw_joint: limit lower=-2.3 upper=2.3 effort=20 velocity=20 -> lower=-2.3 upper=2.3 effort=17 velocity=87
- joint torso_joint: limit lower=-3 upper=3 effort=300 velocity=12 -> lower=-3 upper=3 effort=300 velocity=11

Commit message: update lus2 knee and ankle_roll

File: lus2/urdf/lus2_joint21.urdf (robot description, URDF)
Before this commit: robot lus2, 29 links, 28 joints
Links:
- link left_ankle_roll_link: geometry collision box size=0.235 0.073 0.0143; collision sphere radius=0.005
- link left_knee_link: geometry collision box size=0.109 0.095 0.278; visual mesh filename=../meshes/left_knee_link_v1.STL
- link right_ankle_roll_link: geometry collision box size=0.235 0.073 0.0143; collision sphere radius=0.005
- link right_knee_link: geometry collision box size=0.109 0.095 0.278; visual mesh filename=../meshes/right_knee_link_v1.STL

File: lus2/urdf/lus2_joint25.urdf (robot description, URDF)
Before this commit: robot lus2, 29 links, 28 joints
Links:
- link left_ankle_roll_link: geometry collision box size=0.235 0.073 0.0143; collision sphere radius=0.005
- link left_knee_link: geometry collision box size=0.109 0.095 0.278; visual mesh filename=../meshes/left_knee_link_v1.STL
- link right_ankle_roll_link: geometry collision box size=0.235 0.073 0.0143; collision sphere radius=0.005
- link right_knee_link: geometry collision box size=0.109 0.095 0.278; visual mesh filename=../meshes/right_knee_link_v1.STL

File: lus2/urdf/lus2_joint27.urdf (robot description, URDF)
Before this commit: robot lus2, 29 links, 28 joints
Links:
- link left_ankle_roll_link: geometry collision box size=0.235 0.073 0.0143; collision sphere radius=0.005
- link left_knee_link: geometry collision box size=0.109 0.095 0.278; visual mesh filename=../meshes/left_knee_link_v1.STL
- link right_ankle_roll_link: geometry collision box size=0.235 0.073 0.0143; collision sphere radius=0.005
- link right_knee_link: geometry collision box size=0.109 0.095 0.278; visual mesh filename=../meshes/right_knee_link_v1.STL
