Commit message: update lus2 knee and ankle_roll STL

File: lus2/urdf/lus2_joint21_relative_imu.urdf (robot description, URDF)
Before this commit: robot lus2, 29 links, 28 joints
Joints:
- joint left_wrist_pitch_joint: type revolute -> fixed
- joint left_wrist_roll_joint: type revolute -> fixed
- joint left_wrist_yaw_joint: type revolute -> fixed
- joint right_wrist_pitch_joint: type revolute -> fixed
- joint right_wrist_roll_joint: type revolute -> fixed
- joint right_wrist_yaw_joint: type revolute -> fixed

File: lus2/urdf/lus2_joint25_relative_imu.urdf (robot description, URDF)
Before this commit: robot lus2, 29 links, 28 joints
Joints:
- joint left_wrist_roll_joint: type revolute -> fixed
- joint right_wrist_roll_joint: type revolute -> fixed
