Commit message: add lumos logo

File: lus2/urdf/lus2.urdf (robot description, URDF)
Before this commit: robot lus2, 29 links, 28 joints
Links:
- link left_ankle_pitch_link: geometry collision mesh filename=../meshes/left_ankle_pitch_link.STL; visual mesh filename=../meshes/left_ankle_pitch_link.STL
- link left_hip_pitch_link: geometry collision mesh filename=../meshes/left_hip_pitch_link.STL; visual mesh filename=../meshes/left_hip_pitch_link.STL
- link left_hip_roll_link: geometry collision mesh filename=../meshes/left_hip_roll_link.STL; visual mesh filename=../meshes/left_hip_roll_link.STL
- link left_hip_yaw_link: geometry collision mesh filename=../meshes/left_hip_yaw_link.STL; visual mesh filename=../meshes/left_hip_yaw_link.STL
- link left_knee_link: geometry collision mesh filename=../meshes/left_knee_link.STL; visual mesh filename=../meshes/left_knee_link_v1.STL
- link right_hip_pitch_link: geometry collision mesh filename=../meshes/right_hip_pitch_link.STL; visual mesh filename=../meshes/right_hip_pitch_link.STL
- link right_hip_roll_link: geometry collision mesh filename=../meshes/right_hip_roll_link.STL; visual mesh filename=../meshes/right_hip_roll_link.STL
- link right_hip_yaw_link: geometry collision mesh filename=../meshes/right_hip_yaw_link.STL; visual mesh filename=../meshes/right_hip_yaw_link.STL
- link right_knee_link: geometry collision mesh filename=../meshes/right_knee_link.STL; visual mesh filename=../meshes/right_knee_link_v1.STL
- link torso_link: geometry collision mesh filename=../meshes/torso_link.STL; visual mesh filename=../meshes/logo1_link.STL
Joints:
- joint head_joint: type fixed -> revolute

File: lus2/urdf/lus2_joint27.urdf (robot description, URDF)
Before this commit: robot lus2, 29 links, 28 joints
Links:
- link left_ankle_pitch_link: geometry collision mesh filename=../meshes/left_ankle_pitch_link.STL; visual mesh filename=../meshes/left_ankle_pitch_link.STL
- link left_hip_pitch_link: geometry collision mesh filename=../meshes/left_hip_pitch_link.STL; visual mesh filename=../meshes/left_hip_pitch_link.STL
- link left_hip_roll_link: geometry collision mesh filename=../meshes/left_hip_roll_link.STL; visual mesh filename=../meshes/left_hip_roll_link.STL
- link left_hip_yaw_link: geometry collision mesh filename=../meshes/left_hip_yaw_link.STL; visual mesh filename=../meshes/left_hip_yaw_link.STL
- link left_knee_link: geometry collision mesh filename=../meshes/left_knee_link.STL; visual mesh filename=../meshes/left_knee_link_v1.STL
- link right_hip_pitch_link: geometry collision mesh filename=../meshes/right_hip_pitch_link.STL; visual mesh filename=../meshes/right_hip_pitch_link.STL
- link right_hip_roll_link: geometry collision mesh filename=../meshes/right_hip_roll_link.STL; visual mesh filename=../meshes/right_hip_roll_link.STL
- link right_hip_yaw_link: geometry collision mesh filename=../meshes/right_hip_yaw_link.STL; visual mesh filename=../meshes/right_hip_yaw_link.STL
- link right_knee_link: geometry collision mesh filename=../meshes/right_knee_link.STL; visual mesh filename=../meshes/right_knee_link_v1.STL
- link torso_link: geometry collision mesh filename=../meshes/torso_link.STL; visual mesh filename=../meshes/torso_link.STL
Joints:
- joint head_joint: type fixed -> revolute
